Commit message: my_bot update

File: description/robot_core.xacro (robot description, xacro)
@@ -4,12 +4,12 @@
     <xacro:property name="chassis_length" value="0.14"/>
     <xacro:property name="chassis_width" value="0.175"/>
-    <xacro:property name="chassis_height" value="0.08"/>
+    <xacro:property name="chassis_height" value="0.110"/>
     <xacro:property name="chassis_mass" value="1.0"/>
     <xacro:property name="wheel_radius" value="0.034"/>
     <xacro:property name="wheel_thickness" value="0.025"/>
     <xacro:property name="wheel_mass" value="0.02"/>
-    <xacro:property name="wheel_offset_x" value="0.13"/>
-    <xacro:property name="wheel_offset_y" value="0.1"/>
-    <xacro:property name="wheel_offset_z" value="-0.035"/>
+    <xacro:property name="chassis_offset_x" value="0.12"/>
+    <xacro:property name="chassis_offset_y" value="0.1"/>
+    <xacro:property name="chassis_offset_z" value="0.035"/>
     <xacro:property name="caster_wheel_radius" value="0.03"/>
     <xacro:property name="caster_wheel_mass" value="0.04"/>
@@ -44,8 +44,11 @@
     </link>
     <!-- CHASSIS LINK -->
+    <!-- The box origin is at the bottom and back, the chassis relate to base_link is -->
+    <!-- chassic move left by ( ${-wheel_offset_x} ) and move up by ${wheel_offset_z}) -->
+    <!-- relative to the origin <0, 0, 0>-->
     <joint name="chassis_joint" type="fixed">
         <parent link="base_link"/>
         <child link="chassis"/>
-        <origin xyz="${-wheel_offset_x} 0 ${-wheel_offset_z}"/>
+        <origin xyz="${-chassis_offset_x} 0 ${chassis_offset_z}"/>
     </joint>
     <link name="chassis">
@@ -71,8 +74,12 @@
     </gazebo>
     <!-- LEFT WHEEL LINK -->
+    <!-- clockwise==(negative rotation) counterclockwise== (positive rotation)-->
+    <!-- right hand rule -->
+    <!-- axis z is "1", car is moving fordward-->
     <joint name="left_wheel_joint" type="continuous">
         <parent link="base_link"/>
         <child link="left_wheel"/>
-        <origin xyz="0 ${wheel_offset_y} 0" rpy="-${pi/2} 0 0" />
+        <origin xyz="0 ${chassis_offset_y} 0" rpy="-${pi/2} 0 0" />
+       <!--<origin xyz="0 ${chassis_offset_y} 0" rpy="0 0 0" /> -->
         <axis xyz="0 0 1"/>
     </joint>
@@ -100,5 +107,5 @@
         <parent link="base_link"/>
         <child link="right_wheel"/>
-        <origin xyz="0 ${-wheel_offset_y} 0" rpy="${pi/2} 0 0" />
+        <origin xyz="0 ${-chassis_offset_y} 0" rpy="${pi/2} 0 0" />
         <axis xyz="0 0 -1"/>
     </joint>
