Commit message: second commit

File: description/RGBD_camera.xacro (robot description, xacro)
@@ -3,5 +3,5 @@
     <xacro:property name="camera_offset_x" value="0.15"/>
     <xacro:property name="camera_offset_y" value="0.0"/>
-    <xacro:property name="camera_offset_z" value="0.08"/>
+    <xacro:property name="camera_offset_z" value="0.11"/>
     <joint name="camera_joint" type="fixed">
         <parent link="chassis"/>
@@ -25,23 +25,22 @@
     <gazebo reference="camera_link">
         <material>Gazebo/Black</material>
-        <sensor name="camera" type="camera">
-            <pose> 0 0 0 0 0 0 </pose>
-            <visualize>true</visualize>
-            <update_rate>10</update_rate>
+        <sensor name="rgbd_camera" type="rgbd_camera">
             <camera>
-                <camera_info_topic>camera/camera_info</camera_info_topic>
-                <horizontal_fov>1.089</horizontal_fov>
+                <horizontal_fov>1.25</horizontal_fov>
                 <image>
-                    <format>R8G8B8</format>
-                    <width>640</width>
-                    <height>480</height>
+                    <width>320</width>
+                    <height>240</height>
                 </image>
                 <clip>
-                    <near>0.05</near>
-                    <far>8.0</far>
+                    <near>0.3</near>
+                    <far>15</far>
                 </clip>
+                <optical_frame_id>camera_link</optical_frame_id>
             </camera>
-            <topic>camera/image</topic>
-            <gz_frame_id>camera_link_optical</gz_frame_id>
+            <always_on>1</always_on>
+            <update_rate>20</update_rate>
+            <visualize>true</visualize>
+            <topic>camera</topic>
+            <gz_frame_id>camera_link</gz_frame_id>
         </sensor>
     </gazebo>

File: description/gazebo_control.xacro (robot description, xacro)
@@ -2,19 +2,35 @@
 <robot xmlns:xacro="http://www.ros.org/wiki/xacro">
     <gazebo>
-        <plugin name="diff_drive" filename="libgazebo_ros_diff_drive.so">
-            <!-- Wheel Information -->
+        <plugin filename="gz-sim-diff-drive-system" name="gz::sim::systems::DiffDrive">
+             <!-- Input -->
+            <topic>cmd_vel</topic>
+            <!-- Wheel joints -->
             <left_joint>left_wheel_joint</left_joint>
             <right_joint>right_wheel_joint</right_joint>
-            <wheel_separation>0.18</wheel_separation>
-            <wheel_diameter>0.072</wheel_diameter>
-            <!-- Limits -->
-            <max_wheel_torque>200</max_wheel_torque>
-            <max_wheel_acceleration>10.0</max_wheel_acceleration>
+            <!-- Wheel parameters -->
+            <wheel_separation>0.1</wheel_separation>
+            <wheel_radius>0.034</wheel_radius>
+            <!-- Control gains and limits (optional) -->
+            <max_velocity>3.0</max_velocity>
+            <max_linear_acceleration>1</max_linear_acceleration>
+            <min_linear_acceleration>-1</min_linear_acceleration>
+            <max_angular_acceleration>2</max_angular_acceleration>
+            <min_angular_acceleration>-2</min_angular_acceleration>
+            <max_linear_velocity>0.5</max_linear_velocity>
+            <min_linear_velocity>-0.5</min_linear_velocity>
+            <max_angular_velocity>1</max_angular_velocity>
+            <min_angular_velocity>-1</min_angular_velocity>
             <!-- Output -->
-            <odometry_frame>odom</odometry_frame>
-            <robot_base_frame>base_link</robot_base_frame>
-            <publish_odom>true</publish_odom>
-            <publish_odom_tf>true</publish_odom_tf>
-            <publish_wheel_tf>true</publish_wheel_tf>
+            <odom_topic>odom</odom_topic>
+            <tf_topic>/tf</tf_topic>
+            <frame_id>odom</frame_id>
+            <child_frame_id>base_footprint</child_frame_id>
+            <odom_publisher_frequency>30</odom_publisher_frequency>
+        </plugin>
+        <plugin filename="gz-sim-joint-state-publisher-system"
+            name="gz::sim::systems::JointStatePublisher">
+            <topic>joint_states</topic>
+            <joint_name>left_wheel_joint</joint_name>
+            <joint_name>right_wheel_joint</joint_name>
         </plugin>
     </gazebo>

File: description/lidar.xacro (robot description, xacro)
@@ -1,8 +1,12 @@
 <?xml version="1.0"?>
 <robot xmlns:xacro="http://www.ros.org/wiki/xacro" >
+    <xacro:property name="laser_offset_x" value="0.07"/>
+    <xacro:property name="laser_offset_y" value="0.0"/>
+    <xacro:property name="laser_offset_z" value="0.15"/>
+    <xacro:property name="laser_offset_yaw" value="1.5708"/>
     <joint name="laser_joint" type="fixed">
         <parent link="chassis"/>
         <child link="laser_frame"/>
-        <origin xyz="0.1 0 0.12" rpy="0 0 0"/>
+        <origin xyz="${laser_offset_x} ${laser_offset_y} ${laser_offset_z}" rpy="0 0 -${laser_offset_yaw}"/>
     </joint>
     <link name="laser_frame">
@@ -31,9 +35,9 @@
     <gazebo reference="laser_frame">
         <material>Gazebo/Black</material>
-        <sensor name="laser" type="ray">
+        <sensor name="laser" type="gpu_lidar">
             <pose> 0 0 0 0 0 0 </pose>
             <visualize>false</visualize>
             <update_rate>10</update_rate>
-            <ray>
+            <lidar>
                 <scan>
                     <horizontal>
@@ -47,12 +51,7 @@
                     <max>12</max>
                 </range>
-            </ray>
-            <plugin name="laser_controller" filename="libgazebo_ros_ray_sensor.so">
-                <ros>
-                    <argument>~/out:=scan</argument>
-                </ros>
-                <output_type>sensor_msgs/LaserScan</output_type>
-                <frame_name>laser_frame</frame_name>
-            </plugin>
+            </lidar>
+            <topic>scan</topic>
+            <gz_frame_id>laser_frame</gz_frame_id>
         </sensor>
     </gazebo>

File: description/robot_core_skid.xacro (robot description, xacro)
@@ -9,5 +9,5 @@
     <xacro:property name="wheel_thickness" value="0.025"/>
     <xacro:property name="wheel_mass" value="0.02"/>
-    <xacro:property name="chassis_offset_x" value="0.12"/>
+    <xacro:property name="chassis_offset_x" value="0.07"/>
     <xacro:property name="wheel_offset_y" value="0.1"/>
     <xacro:property name="chassis_offset_z" value="0.035"/>
@@ -77,11 +77,62 @@
     <!-- right hand rule -->
     <!-- axis z is "1", car is moving fordward-->
-    <joint name="left_wheel_joint" type="continuous">
+    <joint name="front_left_wheel_joint" type="continuous">
+        <origin xyz="0.05 ${wheel_offset_y} 0" rpy="-${pi/2} 0 0" />
         <parent link="base_link"/>
-        <child link="left_wheel"/>
-        <origin xyz="0 ${wheel_offset_y} 0" rpy="-${pi/2} 0 0" />
+        <child link="front_left_wheel"/>
         <axis xyz="0 0 1"/>
     </joint>
-    <link name="left_wheel">
+    <link name="front_left_wheel">
+        <visual name='front_left_wheel_visual'>
+            <geometry>
+                <cylinder radius="${wheel_radius}" length="${wheel_thickness}"/>
+            </geometry>
+            <material name="blue"/>
+        </visual>
+        <collision>
+            <geometry>
+                <sphere radius="${wheel_radius}"/>
+            </geometry>
+        </collision>
+        <xacro:inertial_cylinder mass="${wheel_mass}" length="${wheel_thickness}" radius="${wheel_radius}">
+            <origin xyz="0 0 0" rpy="0 0 0"/>
+        </xacro:inertial_cylinder>
+    </link>
+     <joint name="rear_left_wheel_joint" type="continuous">
+        <origin xyz="-0.05 ${wheel_offset_y} 0" rpy="-${pi/2} 0 0" />
+        <parent link="base_link"/>
+        <child link="front_left_wheel"/>
+        <axis xyz="0 0 1"/>
+    </joint>
+    <link name="rear_left_wheel">
+        <visual name='rear_left_wheel_visual'>
+            <geometry>
+                <cylinder radius="${wheel_radius}" length="${wheel_thickness}"/>
+            </geometry>
+            <material name="blue"/>
+        </visual>
+        <collision>
+            <geometry>
+                <sphere radius="${wheel_radius}"/>
+            </geometry>
+        </collision>
+        <xacro:inertial_cylinder mass="${wheel_mass}" length="${wheel_thickness}" radius="${wheel_radius}">
+            <origin xyz="0 0 0" rpy="0 0 0"/>
+        </xacro:inertial_cylinder>
+    </link>
+    <gazebo reference="front_left_wheel">
+        <material>Gazebo/Blue</material>
+    </gazebo>
+    <gazebo reference="rear_left_wheel">
+        <material>Gazebo/Blue</material>
+    </gazebo>
+    <!-- RIGHT WHEEL LINK -->
+    <joint name="front_right_wheel_joint" type="continuous">
+        <origin xyz="0.05 ${-wheel_offset_y} 0" rpy="${pi/2} 0 0" />
+        <parent link="base_link"/>
+        <child link="front_right_wheel"/>
+        <axis xyz="0 0 -1"/>
+    </joint>
+    <link name="front_right_wheel">
         <visual>
             <geometry>
@@ -99,15 +150,11 @@
         </xacro:inertial_cylinder>
     </link>
-    <gazebo reference="left_wheel">
-        <material>Gazebo/Blue</material>
-    </gazebo>
-    <!-- RIGHT WHEEL LINK -->
-    <joint name="right_wheel_joint" type="continuous">
+    <joint name="rear_right_wheel_joint" type="continuous">
+        <origin xyz="-0.05 ${-wheel_offset_y} 0" rpy="${pi/2} 0 0" />
         <parent link="base_link"/>
-        <child link="right_wheel"/>
-        <origin xyz="0 ${-wheel_offset_y} 0" rpy="${pi/2} 0 0" />
+        <child link="front_right_wheel"/>
         <axis xyz="0 0 -1"/>
     </joint>
-    <link name="right_wheel">
+    <link name="rear_right_wheel">
         <visual>
             <geometry>
@@ -125,33 +172,9 @@
         </xacro:inertial_cylinder>
     </link>
-    <gazebo reference="right_wheel">
+    <gazebo reference="front_right_wheel">
         <material>Gazebo/Blue</material>
     </gazebo>
-    <!-- CASTER WHEEL LINK -->
-    <joint name="caster_wheel_joint" type="fixed">
-        <parent link="chassis"/>
-        <child link="caster_wheel"/>
-        <origin xyz="${caster_wheel_offset_x} 0 ${caster_wheel_offset_z}"/>
-    </joint>
-    <link name="caster_wheel">
-        <visual>
-            <geometry>
-                <sphere radius="${caster_wheel_radius}"/>
-            </geometry>
-            <material name="white"/>
-        </visual>
-        <collision>
-            <geometry>
-                <sphere radius="${caster_wheel_radius}"/>
-            </geometry>
-        </collision>
-        <xacro:inertial_sphere mass="${caster_wheel_mass}" radius="${caster_wheel_radius}">
-            <origin xyz="0 0 0" rpy="0 0 0"/>
-        </xacro:inertial_sphere>
-    </link>
-    <gazebo reference="caster_wheel">
-        <material>Gazebo/White</material>
-        <mu1 value="0.001"/>
-        <mu2 value="0.001"/>
+    <gazebo reference="rear_right_wheel">
+        <material>Gazebo/Blue</material>
     </gazebo>
 </robot>

File: description/ros2_control.xacro (robot description, xacro)
@@ -34,5 +34,5 @@
         <ros2_control name="GazeboSystem" type="system">
             <hardware>
-                <plugin>gazebo_ros2_control/GazeboSystem</plugin>
+                <plugin>gz_ros2_control/GazeboSimSystem</plugin>
             </hardware>
             <joint name="left_wheel_joint">
@@ -55,7 +55,7 @@
     </xacro:if>
     <gazebo>
-        <plugin name="gazebo_ros2_control" filename="libgazebo_ros2_control.so">
-            <parameters>$(find my_bot)/config/my_controllers.yaml</parameters>
-            <!-- <parameters>$(find my_bot)/config/gaz_ros2_ctl_use_sim.yaml</parameters> -->
+     <!-- Joint state publisher -->
+        <plugin filename="gz_ros2_control-system" name="gz_ros2_control::GazeboSimROS2ControlPlugin">
+            <parameters>$(find my_bot)/config/diff_drive_controller.yaml</parameters>
         </plugin>
     </gazebo>
