Commit message: base_footprint correction

File: description/robot.urdf.xacro (robot description, xacro)
@@ -1,5 +1,5 @@
 <?xml version="1.0"?>
 <robot xmlns:xacro="http://www.ros.org/wiki/xacro"  name="robot">
-    <xacro:arg name="use_ros2_control" default="false"/>
+    <xacro:arg name="use_ros2_control" default="true"/>
     <xacro:arg name="sim_mode" default="true"/>
     <xacro:include filename="robot_core.xacro" />

File: description/robot_core.xacro (robot description, xacro)
@@ -32,8 +32,7 @@
         <color rgba="1 0 0 1"/>
     </material>
+     <link name="base_footprint"/>
     <!-- BASE LINK -->
-    <link name="base_link">
-         <pose>0 0 0 0 0 0</pose>
-    </link>
+    <link name="base_link"></link>
     <!-- BASE_FOOTPRINT LINK -->
     <joint name="base_footprint_joint" type="fixed">
@@ -42,5 +41,4 @@
         <origin xyz="0 0 ${wheel_radius}" rpy="0 0 0"/>
     </joint>
-    <link name="base_footprint">  </link>
     <!-- CHASSIS LINK -->
     <!-- The box origin is at the bottom and back, the chassis relate to base_link is -->
